File: dev_board/_autosave-dev_board.kicad_pcb (KiCad board)
At the start: 2 copper layers, 35 parts, among them J1 USB_C_Receptacle_USB2.0_14P, J2 AVR-ISP-6, SW1 RESET, SW2 test, SW3 test, U1 AMS1117-3.3, U2 ATmega32L-8A, U3 CH330N, Y1 ASCO

Commit message: initial commit for wifi board
Parts:
- moved J1 50.2 mm to (187.0, 82.0), turned to 180 degrees
- moved U2 47.0 mm to (188.3, 94.8)
- moved U3 44.0 mm to (177.0, 84.5), turned to -90 degrees
- moved D7 30.5 mm to (178.5, 91.5), turned to -90 degrees
- moved D6 26.7 mm to (175.5, 91.5), turned to 90 degrees
