File: MixedSigBoard/ADC.kicad_sch (KiCad schematic)
At the start: 32 parts

Commit message: -Renumber components to match sheet number -Created PCB Constraints and Set-up
Parts:
- gave numbers to parts that had none: 32

Commit message: Add all footprints
Parts:
- J1: footprint PhilsLab_Footprints_KiCad6:AMPHENOL-BNC-031-5640-1010 -> MixSig_Footprints_KiCad6:AMPHENOL-BNC-031-5640-1010
- U2: footprint PhilsLab_Footprints_KiCad6:VSSOP-10 -> MixSig_Footprints_KiCad6:VSSOP-10
Changed lines of the file:
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@@
 			)
 		)
-		(property "Footprint" "PhilsLab_Footprints_KiCad6:VSSOP-10"
+		(property "Footprint" "MixSig_Footprints_KiCad6:VSSOP-10"
 			(at 130.81 156.21 0)
 			(effects
@@
 			)
 		)
-		(property "Footprint" "PhilsLab_Footprints_KiCad6:AMPHENOL-BNC-031-5640-1010"
+		(property "Footprint" "MixSig_Footprints_KiCad6:AMPHENOL-BNC-031-5640-1010"
 			(at 45.72 62.23 0)
 			(effects

Commit message: Layout w/o Traces for MCU, ADC page
Parts:
- renumbered C1 to C300, C2 to C301, C3 to C302, C4 to C303, C5 to C304, C6 to C305, C7 to C306, C8 to C307, C9 to C308, C10 to C309, C11 to C310, C12 to C311, C13 to C312, C14 to C313, C15 to C314, C16 to C315, D1 to D300, J1 to J300, R1 to R300, R2 to R301, R3 to R302, R4 to R303, R5 to R304, R6 to R305, R7 to R306, R8 to R307, R9 to R308, R10 to R309, U1 to U300, U2 to U301, U3 to U302, U4 to U303

Commit message: updated PCB footprints
Parts:
- J300: footprint MixSig_Footprints_KiCad6:AMPHENOL-BNC-031-5640-1010 -> MixSig_Footprints.pretty:AMPHENOL-BNC-031-5640-1010
- U301: footprint MixSig_Footprints_KiCad6:VSSOP-10 -> MixSig_Footprints.pretty:VSSOP-10
Changed lines of the file:
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@@
 			)
 		)
-		(property "Footprint" "MixSig_Footprints_KiCad6:VSSOP-10"
+		(property "Footprint" "MixSig_Footprints.pretty:VSSOP-10"
 			(at 130.81 156.21 0)
 			(effects
@@
 			)
 		)
-		(property "Footprint" "MixSig_Footprints_KiCad6:AMPHENOL-BNC-031-5640-1010"
+		(property "Footprint" "MixSig_Footprints.pretty:AMPHENOL-BNC-031-5640-1010"
 			(at 45.72 62.23 0)
 			(effects

Commit message: Add missing footprints
Parts:
- U301: footprint MixSig_Footprints.pretty:VSSOP-10 -> MixSig_Footprints:VSSOP-10
Changed lines of the file:
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@@
 			)
 		)
-		(property "Footprint" "MixSig_Footprints.pretty:VSSOP-10"
+		(property "Footprint" "MixSig_Footprints:VSSOP-10"
 			(at 130.81 156.21 0)
 			(effects

Commit message: complete the MixSigPCB
-Created Gerber file and compressed to .zip
-created placement file
-filled all components from Mouser/JLCPCB/Digikey
Parts:
- C300, C301, C304, C305, C311: Manufacturer (none) -> TAIYO YUDEN; Manufacturer Part Number (none) -> MLASL168BB5106MTNB33
- C302, C313, C315: Manufacturer (none) -> KEMET; Manufacturer Part Number (none) -> C0402C151J1GACAUTO
- C303, C306, C307, C308, C309, C314: Manufacturer (none) -> TAIYO YUDEN; Manufacturer Part Number (none) -> LMK105B7104KVHF
- C310, C312: Manufacturer (none) -> KYOCERA AVX; Manufacturer Part Number (none) -> 04025C102KAZ2A
- D300: Manufacturer (none) -> NEXPERIA USA INC.; Manufacturer Part Number (none) -> PESD3V3L1BA,115
- J300: Manufacturer (none) -> AMPHENOL RF; Manufacturer Part Number (none) -> 31-5640-1010

Commit message: complete the MixSigPCB
Parts:
- R300: Manufacturer (none) -> UNI-ROYAL(Uniroyal Elec); Manufacturer Part Number (none) -> 0402WGF499JTCE
- R301, R308, R309: Manufacturer (none) -> UNI-ROYAL(Uniroyal Elec); Manufacturer Part Number (none) -> 0402WGF1001TCE
- R302, R303: Manufacturer (none) -> YAGEO; Manufacturer Part Number (none) -> RC0402FR-072M2L
- R304: Manufacturer (none) -> UNI-ROYAL(Uniroyal Elec); Manufacturer Part Number (none) -> 0402WGF6801TCE
- R305: Manufacturer (none) -> UNI-ROYAL(Uniroyal Elec); Manufacturer Part Number (none) -> 0402WGF0000TCE
- R306: Manufacturer (none) -> UNI-ROYAL(Uniroyal Elec); Manufacturer Part Number (none) -> 0402WGJ0223TCE
- R307: Manufacturer (none) -> UNI-ROYAL(Uniroyal Elec); Manufacturer Part Number (none) -> 0402WGJ0123TCE
- U300: Manufacturer (none) -> TEXAS INSTRUMENTS; Manufacturer Part Number (none) -> REF3033AIDBZT
- U301: Manufacturer (none) -> TEXAS INSTRUMENTS; Manufacturer Part Number (none) -> ADC141S626CIMM/NOPB
- U302, U303: Manufacturer (none) -> MICROCHIP; Manufacturer Part Number (none) -> MCP6001T-E/OT
