File: MixedSigBoard/MCU.kicad_sch (KiCad schematic)
At the start: 40 parts

Commit message: -Renumber components to match sheet number -Created PCB Constraints and Set-up
Parts:
- gave numbers to parts that had none: 40

Commit message: Add all footprints
Parts:
- L2: footprint PhilsLab_Footprints_KiCad6:CMC-1206 -> MixSig_Footprints_KiCad6:CMC-1206
Changed lines of the file:
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@@
 			)
 		)
-		(property "Footprint" "PhilsLab_Footprints_KiCad6:CMC-1206"
+		(property "Footprint" "MixSig_Footprints_KiCad6:CMC-1206"
 			(at 222.25 125.73 0)
 			(effects

Commit message: Layout w/o Traces for MCU, ADC page
Parts:
- renumbered C24 to C200, C25 to C201, C26 to C202, C27 to C203, C28 to C204, C29 to C205, C30 to C206, C31 to C207, C32 to C208, C33 to C209, C34 to C210, C35 to C211, C36 to C212, D3 to D200, D4 to D201, D5 to D202, D6 to D203, D7 to D204, D8 to D205, J3 to J200, J4 to J201, L1 to L200, L2 to L201, R17 to R200, R18 to R201, R19 to R202, R20 to R203, R21 to R204, R22 to R205, R23 to R206, R24 to R207, R25 to R208, R26 to R209, R27 to R210, R28 to R211, R29 to R212, R30 to R213, U7 to U200, U8 to U201, Y1 to Y200

Commit message: updated PCB footprints
Parts:
- L201: footprint MixSig_Footprints_KiCad6:CMC-1206 -> MixSig_Footprints.pretty:CMC-1206
Changed lines of the file:
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@@
 			)
 		)
-		(property "Footprint" "MixSig_Footprints_KiCad6:CMC-1206"
+		(property "Footprint" "MixSig_Footprints.pretty:CMC-1206"
 			(at 222.25 125.73 0)
 			(effects

Commit message: add DAC routing, power routing, finish routing
- finished routing, cleared up most DRC errors
- Removed reference designators on F. Silkscreen
Connections:
- net TIM4_CH1: now also R202.1; no longer R201.1
- net TIM4_CH2: now also R201.1; no longer R202.1
Changed lines of the file:
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@@
-		)
-	)
-	(label "TIM4_CH2"
-		(at 19.05 170.18 0)
-		(effects
-			(font
-				(size 1.27 1.27)
-			)
-			(justify left bottom)
 		)
 	)
@@
 		)
 	)
+	(label "TIM4_CH1"
+		(at 19.05 170.18 0)
+		(effects
+			(font
+				(size 1.27 1.27)
+			)
+			(justify left bottom)
+		)
+	)
+	(label "TIM4_CH2"
+		(at 19.05 165.1 0)
+		(effects
+			(font
+				(size 1.27 1.27)
+			)
+			(justify left bottom)
+		)
+	)
 	(label "SWCLK"
 		(at 168.91 163.83 180)
@@
 		(effects
 			(font
-				(size 1.27 1.27)
-			)
-			(justify left bottom)
-		)
-	)
-	(label "TIM4_CH1"
-		(at 19.05 165.1 0)
-		(effects
-			(font

Commit message: complete the MixSigPCB
-Created Gerber file and compressed to .zip
-created placement file
-filled all components from Mouser/JLCPCB/Digikey
Parts:
- C200: Manufacturer (none) -> TAIYO YUDEN; Manufacturer Part Number (none) -> MLASL168BB5106MTNB33
- C201, C205: Manufacturer (none) -> KYOCERA AVX; Manufacturer Part Number (none) -> KAM05ACG1H100JH
- C202, C203, C204, C206, C207, C210, C212: Manufacturer (none) -> TAIYO YUDEN; Manufacturer Part Number (none) -> LMK105B7104KVHF
- C208: Manufacturer (none) -> MURATA ELECTRONICS; Manufacturer Part Number (none) -> GRM022C81C103ME01L
- C209, C211: Manufacturer (none) -> YAGEO; Manufacturer Part Number (none) -> CC0603KRX5R6BB105
- D200: Manufacturer (none) -> TT ELECTRONICS/OPTEK TECHNOLOGY; Manufacturer Part Number (none) -> OVSARGB4R8
- D201, D202, D203, D204, D205: Manufacturer (none) -> NEXPERIA USA INC.; Manufacturer Part Number (none) -> PESD3V3L1BA,115
- J200: Manufacturer (none) -> CNC TECH; Manufacturer Part Number (none) -> 3220-10-0100-00
- J201: Manufacturer (none) -> Korean Hroparts Elec; Manufacturer Part Number (none) -> TYPE-C-31-M-12
- L200: Manufacturer (none) -> MURATA ELECTRONICS; Manufacturer Part Number (none) -> BLM15BX601SZ1D

Commit message: complete the MixSigPCB
Parts:
- L201: Manufacturer (none) -> HYHONGYEX; Manufacturer Part Number (none) -> CMF3216F-900-2P-T
- R200, R201, R202: Manufacturer (none) -> UNI-ROYAL(Uniroyal Elec); Manufacturer Part Number (none) -> 0402WGF1001TCE
- R203, R204, R206: Manufacturer (none) -> UNI-ROYAL(Uniroyal Elec); Manufacturer Part Number (none) -> 0402WGF1002TCE
- R205: Manufacturer (none) -> UNI-ROYAL(Uniroyal Elec); Manufacturer Part Number (none) -> 0402WGF0000TCE
- R207, R208, R209, R210: Manufacturer (none) -> UNI-ROYAL(Uniroyal Elec); Manufacturer Part Number (none) -> 0402WGF499JTCE
- R211: Manufacturer (none) -> UNI-ROYAL(Uniroyal Elec); Manufacturer Part Number (none) -> 0402WGF1501TCE
- R212, R213: Manufacturer (none) -> UNI-ROYAL(Uniroyal Elec); Manufacturer Part Number (none) -> 0402WGF5101TCE
- U201: Manufacturer (none) -> STMicroelectronics; Manufacturer Part Number (none) -> USBLC6-2SC6
- Y200: Manufacturer (none) -> Epson Timing; Manufacturer Part Number (none) -> TSX-3225 16.0000MF09Z-AC3
