File: MixedSigBoard/Power.kicad_sch (KiCad schematic)
At the start: 21 parts

Commit message: Change Buck Inductor
Parts:
- L4: renamed from L?; value 15u -> 68u
- gave numbers to parts that had none: 20
Other:
- company: Phil's Lab -> Austin Adam
- title: Mixed-Signal Demo PCB -> Mixed-Signal PCB

Commit message: -Renumber components to match sheet number -Created PCB Constraints and Set-up
Parts:
- renumbered C1 to C37, C45 to C38, C38 to C39, C39 to C40, C40 to C41, C41 to C42, C42 to C43, C43 to C44, C44 to C45, L1 to L3, R1 to R31
Changed lines of the file:
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@@
 	(wire
 		(pts
-			(xy 34.29 59.69) (xy 34.29 60.96)
+			(xy 34.29 58.42) (xy 34.29 60.96)
 		)
 		(stroke
@@
 		(on_board yes)
 		(dnp no)
-		(property "Reference" "#PWR057"
+		(property "Reference" "#PWR0105"
 			(at 114.3 83.82 0)
 			(effects
@@
 			(project "Power"
 				(path "/c49d23ab-146d-4089-864f-2d22b5b414b9/00000000-0000-0000-0000-000061c5cb7e"
-					(reference "#PWR057")
+					(reference "#PWR0105")
 					(unit 1)
 				)
@@
 		(on_board yes)
 		(dnp no)
-		(property "Reference" "#PWR067"
+		(property "Reference" "#PWR0115"
 			(at 270.51 72.39 0)
 			(effects
@@
 			(project "Power"
 				(path "/c49d23ab-146d-4089-864f-2d22b5b414b9/00000000-0000-0000-0000-000061c5cb7e"
-					(reference "#PWR067")
+					(reference "#PWR0115")
 					(unit 1)
 				)
@@
 		(on_board yes)
 		(dnp no)
-		(property "Reference" "#PWR060"
+		(property "Reference" "#PWR0108"
 			(at 163.83 113.03 0)
 			(effects
@@
 			(project "Power"
 				(path "/c49d23ab-146d-4089-864f-2d22b5b414b9/00000000-0000-0000-0000-000061c5cb7e"
-					(reference "#PWR060")
+					(reference "#PWR0108")
 					(unit 1)
 				)
@@
 		(on_board yes)
 		(dnp no)
-		(property "Reference" "#PWR055"
+		(property "Reference" "#PWR0103"
 			(at 62.23 63.5 0)
 			(effects
@@
 			(project "Power"
 				(path "/c49d23ab-146d-4089-864f-2d22b5b414b9/00000000-0000-0000-0000-000061c5cb7e"
-					(reference "#PWR055")
+					(reference "#PWR0103")
 					(unit 1)
 				)
@@
 		(on_board yes)
 		(dnp no)
-		(property "Reference" "#PWR058"
+		(property "Reference" "#PWR0106"
 			(at 130.81 63.5 0)
 			(effects
@@
 			(project "Power"
 				(path "/c49d23ab-146d-4089-864f-2d22b5b414b9/00000000-0000-0000-0000-000061c5cb7e"
-					(reference "#PWR058")
+					(reference "#PWR0106")
 					(unit 1)
 				)
@@
 		(on_board yes)
 		(dnp no)
-		(property "Reference" "C39"
+		(property "Reference" "C40"
 			(at 101.6 66.04 0)
 			(effects
@@
 			(project "Power"
 				(path "/c49d23ab-146d-4089-864f-2d22b5b414b9/00000000-0000-0000-0000-000061c5cb7e"
-					(reference "C39")
+					(reference "C40")
 					(unit 1)
 				)
@@
 		(on_board yes)
 		(dnp no)
-		(property "Reference" "C40"
+		(property "Reference" "C41"
 			(at 134.62 66.04 0)
 			(effects
@@
 			(project "Power"
 				(path "/c49d23ab-146d-4089-864f-2d22b5b414b9/00000000-0000-0000-0000-000061c5cb7e"
-					(reference "C40")
+					(reference "C41")
 					(unit 1)
 				)
@@
 	(symbol
 		(lib_id "power:VBUS")
-		(at 34.29 59.69 0)
+		(at 34.29 58.42 0)
 		(unit 1)
 		(exclude_from_sim no)
@@
 		(on_board yes)
 		(dnp no)
-		(property "Reference" "#PWR052"
-			(at 34.29 63.5 0)
+		(property "Reference" "#PWR0100"
+			(at 34.29 62.23 0)
 			(effects
 				(font
@@
 		)
 		(property "Value" "VBUS"
-			(at 34.29 55.88 0)
+			(at 34.29 54.61 0)
 			(effects
 				(font
@@
 		)
 		(property "Footprint" ""
-			(at 34.29 59.69 0)
+			(at 34.29 58.42 0)
 			(effects
 				(font
@@
 		)
 		(property "Datasheet" ""
-			(at 34.29 59.69 0)
+			(at 34.29 58.42 0)
 			(effects
 				(font
@@
 		)
 		(property "Description" ""
-			(at 34.29 59.69 0)
+			(at 34.29 58.42 0)
 			(effects
 				(font
@@
 			(project "Power"
 				(path "/c49d23ab-146d-4089-864f-2d22b5b414b9/00000000-0000-0000-0000-000061c5cb7e"
-					(reference "#PWR052")
+					(reference "#PWR0100")
 					(unit 1)
 				)
@@
 		(on_board yes)
 		(dnp no)
-		(property "Reference" "C1"
+		(property "Reference" "C37"
 			(at 43.18 66.04 0)
 			(effects
@@
 			(project "Power"
 				(path "/c49d23ab-146d-4089-864f-2d22b5b414b9/00000000-0000-0000-0000-000061c5cb7e"
-					(reference "C1")
+					(reference "C37")
 					(unit 1)
 				)
@@
 		(on_board yes)
 		(dnp no)
-		(property "Reference" "C45"
+		(property "Reference" "C38"
 			(at 68.58 66.04 0)
 			(effects
@@
 			(project "Power"
 				(path "/c49d23ab-146d-4089-864f-2d22b5b414b9/00000000-0000-0000-0000-000061c5cb7e"
-					(reference "C45")
+					(reference "C38")
 					(unit 1)
 				)
@@
 		(on_board yes)
 		(dnp no)
-		(property "Reference" "#PWR053"
+		(property "Reference" "#PWR0101"
 			(at 34.29 80.01 0)
 			(effects
@@
 			(project "Power"
 				(path "/c49d23ab-146d-4089-864f-2d22b5b414b9/00000000-0000-0000-0000-000061c5cb7e"
-					(reference "#PWR053")
+					(reference "#PWR0101")
 					(unit 1)
 				)
@@
 		(on_board yes)
 		(dnp no)
-		(property "Reference" "#PWR054"
+		(property "Reference" "#PWR0102"
 			(at 59.69 80.01 0)
 			(effects
@@
 			(project "Power"
 				(path "/c49d23ab-146d-4089-864f-2d22b5b414b9/00000000-0000-0000-0000-000061c5cb7e"
-					(reference "#PWR054")
+					(reference "#PWR0102")
 					(unit 1)
 				)
@@
 		(on_board yes)
 		(dnp no)
-		(property "Reference" "R1"
+		(property "Reference" "R31"
 			(at 91.44 54.61 90)
 			(effects
@@
 			(project "Power"
 				(path "/c49d23ab-146d-4089-864f-2d22b5b414b9/00000000-0000-0000-0000-000061c5cb7e"
-					(reference "R1")
+					(reference "R31")
 					(unit 1)
 				)
@@
 		(on_board yes)
 		(dnp no)
-		(property "Reference" "C44"
+		(property "Reference" "C45"
 			(at 240.03 54.61 90)
 			(effects
@@
 			(project "Power"
 				(path "/c49d23ab-146d-4089-864f-2d22b5b414b9/00000000-0000-0000-0000-000061c5cb7e"
-					(reference "C44")
+					(reference "C45")
 					(unit 1)
 				)
@@
 		(on_board yes)
 		(dnp no)
-		(property "Reference" "#PWR066"
+		(property "Reference" "#PWR0114"
 			(at 251.46 85.09 0)
 			(effects
@@
 			(project "Power"
 				(path "/c49d23ab-146d-4089-864f-2d22b5b414b9/00000000-0000-0000-0000-000061c5cb7e"
-					(reference "#PWR066")
+					(reference "#PWR0114")
 					(unit 1)
 				)
@@
 		(on_board yes)
 		(dnp no)
-		(property "Reference" "#PWR064"
+		(property "Reference" "#PWR0112"
 			(at 234.95 64.77 0)
 			(effects
@@
 			(project "Power"
 				(path "/c49d23ab-146d-4089-864f-2d22b5b414b9/00000000-0000-0000-0000-000061c5cb7e"
-					(reference "#PWR064")
+					(reference "#PWR0112")
 					(unit 1)
 				)
@@
 		(on_board yes)
 		(dnp no)
-		(property "Reference" "#PWR065"
+		(property "Reference" "#PWR0113"
 			(at 251.46 60.96 0)
 			(effects
@@
 			(project "Power"
 				(path "/c49d23ab-146d-4089-864f-2d22b5b414b9/00000000-0000-0000-0000-000061c5cb7e"
-					(reference "#PWR065")
+					(reference "#PWR0113")
 					(unit 1)
 				)
@@
 		(on_board yes)
 		(dnp no)
-		(property "Reference" "#PWR062"
+		(property "Reference" "#PWR0110"
 			(at 220.98 60.96 0)
 			(effects
@@
 			(project "Power"
 				(path "/c49d23ab-146d-4089-864f-2d22b5b414b9/00000000-0000-0000-0000-000061c5cb7e"
-					(reference "#PWR062")
+					(reference "#PWR0110")
 					(unit 1)
 				)
@@
 		(on_board yes)
 		(dnp no)
-		(property "Reference" "C43"
+		(property "Reference" "C44"
 			(at 236.22 71.12 0)
 			(effects
@@
 			(project "Power"
 				(path "/c49d23ab-146d-4089-864f-2d22b5b414b9/00000000-0000-0000-0000-000061c5cb7e"
-					(reference "C43")
+					(reference "C44")
 					(unit 1)
 				)
@@
 		(on_board yes)
 		(dnp no)
-		(property "Reference" "#PWR063"
+		(property "Reference" "#PWR0111"
 			(at 220.98 85.09 0)
 			(effects
@@
 			(project "Power"
 				(path "/c49d23ab-146d-4089-864f-2d22b5b414b9/00000000-0000-0000-0000-000061c5cb7e"
-					(reference "#PWR063")
+					(reference "#PWR0111")
 					(unit 1)
 				)
@@
 		(on_board yes)
 		(dnp no)
-		(property "Reference" "C41"
+		(property "Reference" "C42"
 			(at 134.62 116.84 0)
 			(effects
@@
 			(project "Power"
 				(path "/c49d23ab-146d-4089-864f-2d22b5b414b9/00000000-0000-0000-0000-000061c5cb7e"
-					(reference "C41")
+					(reference "C42")
 					(unit 1)
 				)
@@
 		(on_board yes)
 		(dnp no)
-		(property "Reference" "#PWR056"
+		(property "Reference" "#PWR0104"
 			(at 97.79 135.89 0)
 			(effects
@@
 			(project "Power"
 				(path "/c49d23ab-146d-4089-864f-2d22b5b414b9/00000000-0000-0000-0000-000061c5cb7e"
-					(reference "#PWR056")
+					(reference "#PWR0104")
 					(unit 1)
 				)
@@
 		(on_board yes)
 		(dnp no)
-		(property "Reference" "C38"
+		(property "Reference" "C39"
 			(at 76.2 116.84 0)
 			(effects
@@
 			(project "Power"
 				(path "/c49d23ab-146d-4089-864f-2d22b5b414b9/00000000-0000-0000-0000-000061c5cb7e"
-					(reference "C38")
+					(reference "C39")
 					(unit 1)
 				)
@@
 		(on_board yes)
 		(dnp no)
-		(property "Reference" "C42"
+		(property "Reference" "C43"
 			(at 165.1 116.84 0)
 			(effects
@@
 			(project "Power"
 				(path "/c49d23ab-146d-4089-864f-2d22b5b414b9/00000000-0000-0000-0000-000061c5cb7e"
-					(reference "C42")
+					(reference "C43")
 					(unit 1)
 				)
@@
 		(on_board yes)
 		(dnp no)
-		(property "Reference" "#PWR059"
+		(property "Reference" "#PWR0107"
 			(at 148.59 144.78 0)
 			(effects
@@
 			(project "Power"
 				(path "/c49d23ab-146d-4089-864f-2d22b5b414b9/00000000-0000-0000-0000-000061c5cb7e"
-					(reference "#PWR059")
+					(reference "#PWR0107")
 					(unit 1)
 				)
@@
 		(on_board yes)
 		(dnp no)
-		(property "Reference" "#PWR061"
+		(property "Reference" "#PWR0109"
 			(at 191.77 130.81 0)
 			(effects
@@
 			(project "Power"
 				(path "/c49d23ab-146d-4089-864f-2d22b5b414b9/00000000-0000-0000-0000-000061c5cb7e"
-					(reference "#PWR061")
+					(reference "#PWR0109")
 					(unit 1)
 				)
@@
 		(dnp no)
 		(fields_autoplaced yes)
-		(property "Reference" "L1"
+		(property "Reference" "L3"
 			(at 46.99 55.88 90)
 			(effects
@@
 			(project "Power"
 				(path "/c49d23ab-146d-4089-864f-2d22b5b414b9/00000000-0000-0000-0000-000061c5cb7e"
-					(reference "L1")
+					(reference "L3")
 					(unit 1)
 				)

Commit message: Add all footprints
Parts:
- L4: footprint PhilsLab_Footprints_KiCad6:MWSA0603S -> MixSig_Footprints_KiCad6:MWSA0603S
Changed lines of the file:
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@@
 			)
 		)
-		(property "Footprint" "PhilsLab_Footprints_KiCad6:MWSA0603S"
+		(property "Footprint" "MixSig_Footprints_KiCad6:MWSA0603S"
 			(at 119.38 111.76 0)
 			(effects

Commit message: Layout w/o Traces for MCU, ADC page
Parts:
- renumbered C37 to C100, C38 to C101, C39 to C102, C40 to C103, C41 to C104, C42 to C105, C43 to C106, C44 to C107, C45 to C108, D9 to D100, L3 to L100, L4 to L101, R31 to R100, R32 to R101, R33 to R102, R34 to R103, R35 to R104, R36 to R105, U9 to U100, U10 to U101, U11 to U102
Changed lines of the file:
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@@
 		(on_board yes)
 		(dnp no)
-		(property "Reference" "U10"
+		(property "Reference" "U101"
 			(at 114.3 53.34 0)
 			(effects
@@
 			(project "Power"
 				(path "/c49d23ab-146d-4089-864f-2d22b5b414b9/00000000-0000-0000-0000-000061c5cb7e"
-					(reference "U10")
+					(reference "U101")
 					(unit 1)
 				)
@@
 		(on_board yes)
 		(dnp no)
-		(property "Reference" "C40"
+		(property "Reference" "C103"
 			(at 101.6 66.04 0)
 			(effects
@@
 			(project "Power"
 				(path "/c49d23ab-146d-4089-864f-2d22b5b414b9/00000000-0000-0000-0000-000061c5cb7e"
-					(reference "C40")
+					(reference "C103")
 					(unit 1)
 				)
@@
 		(on_board yes)
 		(dnp no)
-		(property "Reference" "C41"
+		(property "Reference" "C104"
 			(at 134.62 66.04 0)
 			(effects
@@
 			(project "Power"
 				(path "/c49d23ab-146d-4089-864f-2d22b5b414b9/00000000-0000-0000-0000-000061c5cb7e"
-					(reference "C41")
+					(reference "C104")
 					(unit 1)
 				)
@@
 		(on_board yes)
 		(dnp no)
-		(property "Reference" "C37"
+		(property "Reference" "C100"
 			(at 43.18 66.04 0)
 			(effects
@@
 			(project "Power"
 				(path "/c49d23ab-146d-4089-864f-2d22b5b414b9/00000000-0000-0000-0000-000061c5cb7e"
-					(reference "C37")
+					(reference "C100")
 					(unit 1)
 				)
@@
 		(on_board yes)
 		(dnp no)
-		(property "Reference" "C38"
+		(property "Reference" "C101"
 			(at 68.58 66.04 0)
 			(effects
@@
 			(project "Power"
 				(path "/c49d23ab-146d-4089-864f-2d22b5b414b9/00000000-0000-0000-0000-000061c5cb7e"
-					(reference "C38")
+					(reference "C101")
 					(unit 1)
 				)
@@
 		(on_board yes)
 		(dnp no)
-		(property "Reference" "R31"
+		(property "Reference" "R100"
 			(at 91.44 54.61 90)
 			(effects
@@
 			(project "Power"
 				(path "/c49d23ab-146d-4089-864f-2d22b5b414b9/00000000-0000-0000-0000-000061c5cb7e"
-					(reference "R31")
+					(reference "R100")
 					(unit 1)
 				)
@@
 		(on_board yes)
 		(dnp no)
-		(property "Reference" "U11"
+		(property "Reference" "U102"
 			(at 252.73 64.77 0)
 			(effects
@@
 			(project "Power"
 				(path "/c49d23ab-146d-4089-864f-2d22b5b414b9/00000000-0000-0000-0000-000061c5cb7e"
-					(reference "U11")
+					(reference "U102")
 					(unit 1)
 				)
@@
 		(on_board yes)
 		(dnp no)
-		(property "Reference" "C45"
+		(property "Reference" "C108"
 			(at 240.03 54.61 90)
 			(effects
@@
 			(project "Power"
 				(path "/c49d23ab-146d-4089-864f-2d22b5b414b9/00000000-0000-0000-0000-000061c5cb7e"
-					(reference "C45")
+					(reference "C108")
 					(unit 1)
 				)
@@
 		(on_board yes)
 		(dnp no)
-		(property "Reference" "R35"
+		(property "Reference" "R104"
 			(at 223.52 60.96 0)
 			(effects
@@
 			(project "Power"
 				(path "/c49d23ab-146d-4089-864f-2d22b5b414b9/00000000-0000-0000-0000-000061c5cb7e"
-					(reference "R35")
+					(reference "R104")
 					(unit 1)
 				)
@@
 		(on_board yes)
 		(dnp no)
-		(property "Reference" "R36"
+		(property "Reference" "R105"
 			(at 223.52 71.12 0)
 			(effects
@@
 			(project "Power"
 				(path "/c49d23ab-146d-4089-864f-2d22b5b414b9/00000000-0000-0000-0000-000061c5cb7e"
-					(reference "R36")
+					(reference "R105")
 					(unit 1)
 				)
@@
 		(on_board yes)
 		(dnp no)
-		(property "Reference" "C44"
+		(property "Reference" "C107"
 			(at 236.22 71.12 0)
 			(effects
@@
 			(project "Power"
 				(path "/c49d23ab-146d-4089-864f-2d22b5b414b9/00000000-0000-0000-0000-000061c5cb7e"
-					(reference "C44")
+					(reference "C107")
 					(unit 1)
 				)
@@
 		(on_board yes)
 		(dnp no)
-		(property "Reference" "U9"
+		(property "Reference" "U100"
 			(at 97.79 104.14 0)
 			(effects
@@
 			(project "Power"
 				(path "/c49d23ab-146d-4089-864f-2d22b5b414b9/00000000-0000-0000-0000-000061c5cb7e"
-					(reference "U9")
+					(reference "U100")
 					(unit 1)
 				)
@@
 		(on_board yes)
 		(dnp no)
-		(property "Reference" "L4"
+		(property "Reference" "L101"
 			(at 119.38 109.22 90)
 			(effects
@@
 			(project "Power"
 				(path "/c49d23ab-146d-4089-864f-2d22b5b414b9/00000000-0000-0000-0000-000061c5cb7e"
-					(reference "L4")
+					(reference "L101")
 					(unit 1)
 				)
@@
 		(on_board yes)
 		(dnp no)
-		(property "Reference" "C42"
+		(property "Reference" "C105"
 			(at 134.62 116.84 0)
 			(effects
@@
 			(project "Power"
 				(path "/c49d23ab-146d-4089-864f-2d22b5b414b9/00000000-0000-0000-0000-000061c5cb7e"
-					(reference "C42")
+					(reference "C105")
 					(unit 1)
 				)
@@
 		(on_board yes)
 		(dnp no)
-		(property "Reference" "R32"
+		(property "Reference" "R101"
 			(at 151.13 116.84 0)
 			(effects
@@
 			(project "Power"
 				(path "/c49d23ab-146d-4089-864f-2d22b5b414b9/00000000-0000-0000-0000-000061c5cb7e"
-					(reference "R32")
+					(reference "R101")
 					(unit 1)
 				)
@@
 		(on_board yes)
 		(dnp no)
-		(property "Reference" "C39"
+		(property "Reference" "C102"
 			(at 76.2 116.84 0)
 			(effects
@@
 			(project "Power"
 				(path "/c49d23ab-146d-4089-864f-2d22b5b414b9/00000000-0000-0000-0000-000061c5cb7e"
-					(reference "C39")
+					(reference "C102")
 					(unit 1)
 				)
@@
 		(on_board yes)
 		(dnp no)
-		(property "Reference" "R33"
+		(property "Reference" "R102"
 			(at 151.13 130.81 0)
 			(effects
@@
 			(project "Power"
 				(path "/c49d23ab-146d-4089-864f-2d22b5b414b9/00000000-0000-0000-0000-000061c5cb7e"
-					(reference "R33")
+					(reference "R102")
 					(unit 1)
 				)
@@
 		(on_board yes)
 		(dnp no)
-		(property "Reference" "C43"
+		(property "Reference" "C106"
 			(at 165.1 116.84 0)
 			(effects
@@
 			(project "Power"
 				(path "/c49d23ab-146d-4089-864f-2d22b5b414b9/00000000-0000-0000-0000-000061c5cb7e"
-					(reference "C43")
+					(reference "C106")
 					(unit 1)
 				)
@@
 		(on_board yes)
 		(dnp no)
-		(property "Reference" "D9"
+		(property "Reference" "D100"
 			(at 173.99 105.41 0)
 			(effects
@@
 			(project "Power"
 				(path "/c49d23ab-146d-4089-864f-2d22b5b414b9/00000000-0000-0000-0000-000061c5cb7e"
-					(reference "D9")
+					(reference "D100")
 					(unit 1)
 				)
@@
 		(on_board yes)
 		(dnp no)
-		(property "Reference" "R34"
+		(property "Reference" "R103"
 			(at 194.31 116.84 0)
 			(effects
@@
 			(project "Power"
 				(path "/c49d23ab-146d-4089-864f-2d22b5b414b9/00000000-0000-0000-0000-000061c5cb7e"
-					(reference "R34")
+					(reference "R103")
 					(unit 1)
 				)
@@
 		(dnp no)
 		(fields_autoplaced yes)
-		(property "Reference" "L3"
+		(property "Reference" "L100"
 			(at 46.99 55.88 90)
 			(effects
@@
 			(project "Power"
 				(path "/c49d23ab-146d-4089-864f-2d22b5b414b9/00000000-0000-0000-0000-000061c5cb7e"
-					(reference "L3")
-					(unit 1)
-				)
+					(reference "L100")
+					(unit 1)
+				)

Commit message: updated PCB footprints
Parts:
- L101: footprint MixSig_Footprints_KiCad6:MWSA0603S -> MixSig_Footprints.pretty:MWSA0603S
Changed lines of the file:
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@@
 			)
 		)
-		(property "Footprint" "MixSig_Footprints_KiCad6:MWSA0603S"
+		(property "Footprint" "MixSig_Footprints.pretty:MWSA0603S"
 			(at 119.38 111.76 0)
 			(effects
